File: black-magic-103rc.kicad_pcb (KiCad board)
At the start: 2 copper layers, 57.9 x 24.2 mm, 64 parts, among them J1 USB_B_Micro, J2 JTAG_SWD_10, J3 UART, J4 SWD_CONN, J5 BOOT0, Q1 DMG1024UV, Q2 DMG1023UV, SW1 SW_SPST, U1 USBLC6-2P6, U2 SN74LVC2T45DCUR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

Commit message: [02-04-1948] start to routing
Parts:
- added C22: 100n, Capacitor_SMD:C_0603_1608Metric_Pad1.08x0.95mm_HandSolder, B.Cu at (127.2, 96.3)
- added J6: PORTC, Connector_PinHeader_1.27mm:PinHeader_1x16_P1.27mm_Horizontal, F.Cu at (166.3, 99.8)
- added P1: USB_C_Plug_USB2.0, Connector_USB:USB_C_Receptacle_GCT_USB4110, B.Cu at (119.2, 89.2)
- added R23: 5k1, Resistor_SMD:R_0805_2012Metric_Pad1.20x1.40mm_HandSolder, B.Cu at (127.2, 94.5)
- added R24: 5k1, Resistor_SMD:R_0805_2012Metric_Pad1.20x1.40mm_HandSolder, B.Cu at (127.2, 83.9)
- moved J4 17.3 mm to (130.6, 98.9)
- moved J3 9.65 mm to (117.9, 98.9)
- moved J1 0.44 mm to (120.4, 88.8)
Connections:
- net Net-(J1-D+) renamed /D+
- net Net-(J1-D-) renamed /D-
- U3 pad 10: unconnected-(U3-PC2-Pad10) -> Net-(J6-Pin_3)
- U3 pad 11: unconnected-(U3-PC3-Pad11) -> Net-(J6-Pin_4)
- U3 pad 2: unconnected-(U3-PC13-Pad2) -> Net-(J6-Pin_14)
- U3 pad 24: unconnected-(U3-PC4-Pad24) -> Net-(J6-Pin_5)
- U3 pad 25: unconnected-(U3-PC5-Pad25) -> Net-(J6-Pin_6)
- U3 pad 3: unconnected-(U3-PC14-Pad3) -> Net-(J6-Pin_15)
- U3 pad 37: unconnected-(U3-PC6-Pad37) -> Net-(J6-Pin_7)
- U3 pad 38: unconnected-(U3-PC7-Pad38) -> Net-(J6-Pin_8)
- U3 pad 39: unconnected-(U3-PC8-Pad39) -> Net-(J6-Pin_9)
- U3 pad 4: unconnected-(U3-PC15-Pad4) -> Net-(J6-Pin_16)
- U3 pad 40: unconnected-(U3-PC9-Pad40) -> Net-(J6-Pin_10)
- U3 pad 51: unconnected-(U3-PC10-Pad51) -> Net-(J6-Pin_11)
- U3 pad 52: unconnected-(U3-PC11-Pad52) -> Net-(J6-Pin_12)
- U3 pad 53: unconnected-(U3-PC12-Pad53) -> Net-(J6-Pin_13)
- U3 pad 8: unconnected-(U3-PC0-Pad8) -> Net-(J6-Pin_1)
- U3 pad 9: unconnected-(U3-PC1-Pad9) -> Net-(J6-Pin_2)
Routing:
- net Net-(J6-Pin_5): track 0.00 -> 62.3 mm, vias 0 -> 6
- net Net-(J6-Pin_6): track 0.00 -> 60.4 mm, vias 0 -> 3
- net ITMS_DIR: track 0.00 -> 53.7 mm, vias 0 -> 4
- net /TRSWO: track 0.00 -> 47.0 mm, vias 0 -> 2
- net GND: track 0.00 -> 40.0 mm, vias 0 -> 15
- net ITDO: track 0.00 -> 38.2 mm, vias 0 -> 2
- net +3.3V: track 0.00 -> 35.9 mm, vias 0 -> 10
- net /BOOT0: track 0.00 -> 33.9 mm, vias 0 -> 1
- net /USB+: track 0.00 -> 33.0 mm, vias 0 -> 2
- net IRST_SENSE: track 0.00 -> 32.6 mm, vias 0 -> 4
- net Net-(SW1-B): track 0.00 -> 32.3 mm, vias 0 -> 2
- net /USB-: track 0.00 -> 29.6 mm, vias 0 -> 2
- net /SWCLK: track 0.00 -> 28.2 mm, vias 0 -> 3
- net VBUS: track 0.00 -> 28.1 mm, vias 0 -> 2
- net /SWDIO: track 0.00 -> 27.1 mm, vias 0 -> 1
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
Commit message: [05-25-1348] generate bom
Parts:
- Q1, Q2: footprint Package_TO_SOT_SMD:SOT-363_SC-70-6_Handsoldering -> Package_TO_SOT_SMD:SOT-563
Changed lines of the file:
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@@
 		)
 	)
-	(footprint "Package_TO_SOT_SMD:SOT-363_SC-70-6_Handsoldering"
+	(footprint "Package_TO_SOT_SMD:SOT-563"
 		(layer "F.Cu")
 		(at 158.725002 94.349999 180)
-		(descr "SOT-363, SC-70-6, Handsoldering")
-		(tags "SOT-363 SC-70-6 Handsoldering")
+		(descr "SOT563")
+		(tags "SOT-563")
 		(property "Reference" "Q2"
-			(at 0 -2.25 180)
+			(at 0 -1.9 180)
 			(layer "F.SilkS")
 			(effects
@@
 		)
 		(property "Value" "DMG1023UV"
-			(at 0 2 180)
-			(layer "F.SilkS")
+			(at 0 1.75 180)
+			(layer "F.Fab")
 			(effects
 				(font
@@
 			)
 		)
-		(property "Footprint" "Package_TO_SOT_SMD:SOT-363_SC-70-6_Handsoldering"
+		(property "Footprint" "Package_TO_SOT_SMD:SOT-563"
 			(at 0 0 180)
 			(unlocked yes)
@@
 		(attr smd)
 		(fp_line
-			(start -0.699999 1.159999)
-			(end 0.699998 1.16)
+			(start 0.65 0.9)
+			(end -0.65 0.9)
 			(stroke
 				(width 0.12)
@@
 		)
 		(fp_line
-			(start -0.710001 -1.160001)
-			(end 0.699999 -1.159999)
+			(start 0.65 -0.9)
+			(end -0.45 -0.9)
 			(stroke
 				(width 0.12)
@@
 		(fp_poly
 			(pts
-				(xy -1.08 -1.109998) (xy -1.32 -1.440001) (xy -0.84 -1.44) (xy -1.08 -1.109998)
+				(xy -0.7 -0.9) (xy -0.98 -0.9) (xy -0.7 -1.18) (xy -0.7 -0.9)
 			)
 			(stroke
@@
 		)
 		(fp_line
-			(start 2.4 1.4)
-			(end 2.4 -1.4)
+			(start 1.35 1.1)
+			(end 1.35 -1.1)
 			(stroke
 				(width 0.05)
@@
 		)
 		(fp_line
-			(start -2.4 1.4)
-			(end 2.4 1.4)
+			(start 1.35 1.1)
+			(end -1.35 1.1)
 			(stroke
 				(width 0.05)
@@
 		)
 		(fp_line
-			(start -2.4 -1.4)
-			(end 2.4 -1.4)
+			(start -1.35 -1.1)
+			(end 1.35 -1.1)
 			(stroke
 				(width 0.05)
@@
 		)
 		(fp_line
-			(start -2.4 -1.4)
-			(end -2.4 1.4)
+			(start -1.35 -1.1)
+			(end -1.35 1.1)
 			(stroke
 				(width 0.05)
@@
 		)
 		(fp_line
-			(start 0.675 1.099999)
-			(end -0.674999 1.1)
+			(start 0.65 0.85)
+			(end 0.65 -0.85)
 			(stroke
 				(width 0.1)
@@
 		)
 		(fp_line
-			(start 0.674999 -1.1)
-			(end 0.675 1.099999)
+			(start 0.65 -0.85)
+			(end -0.3 -0.85)
 			(stroke
 				(width 0.1)
@@
 		)
 		(fp_line
-			(start 0.674999 -1.1)
-			(end -0.175 -1.1)
+			(start -0.65 0.85)
+			(end 0.65 0.85)
 			(stroke
 				(width 0.1)
@@
 		)
 		(fp_line
-			(start -0.175 -1.1)
-			(end -0.674998 -0.599998)
+			(start -0.65 -0.5)
+			(end -0.3 -0.85)
 			(stroke
 				(width 0.1)
@@
 		)
 		(fp_line
-			(start -0.674998 -0.599998)
-			(end -0.674999 1.1)
+			(start -0.65 -0.5)
+			(end -0.65 0.85)
 			(stroke
 				(width 0.1)
@@
 		(fp_text user "${REFERENCE}"
 			(at 0 0 -90)
-			(layer "F.SilkS")
+			(layer "F.Fab")
 			(effects
 				(font
-					(size 0.5 0.5)
-					(thickness 0.075)
+					(size 0.4 0.4)
+					(thickness 0.0625)
 				)
 			)
 		)
 		(pad "1" smd roundrect
-			(at -1.33 -0.65 180)
-			(size 1.5 0.4)
+			(at -0.75 -0.5 180)
+			(size 0.7 0.34)
 			(layers "F.Cu" "F.Paste" "F.Mask")
 			(roundrect_rratio 0.25)
@@
 		)
 		(pad "2" smd roundrect
-			(at -1.330002 0.000001 180)
-			(size 1.5 0.4)
+			(at -0.75 0 180)
+			(size 0.7 0.34)
 			(layers "F.Cu" "F.Paste" "F.Mask")
 			(roundrect_rratio 0.25)
@@
 		)
 		(pad "3" smd roundrect
-			(at -1.329998 0.649999 180)
-			(size 1.5 0.4)
+			(at -0.75 0.5 180)
+			(size 0.7 0.34)
 			(layers "F.Cu" "F.Paste" "F.Mask")
 			(roundrect_rratio 0.25)
@@
 		)
 		(pad "4" smd roundrect
-			(at 1.33 0.65 180)
-			(size 1.5 0.4)
+			(at 0.75 0.5 180)
+			(size 0.7 0.34)
 			(layers "F.Cu" "F.Paste" "F.Mask")
 			(roundrect_rratio 0.25)
@@
 		)
 		(pad "5" smd roundrect
-			(at 1.330002 -0.000001 180)
-			(size 1.5 0.4)
+			(at 0.75 0 180)
+			(size 0.7 0.34)
 			(layers "F.Cu" "F.Paste" "F.Mask")
 			(roundrect_rratio 0.25)
@@
 		)
 		(pad "6" smd roundrect
-			(at 1.329998 -0.649999 180)
-			(size 1.5 0.4)
+			(at 0.75 -0.5 180)
+			(size 0.7 0.34)
 			(layers "F.Cu" "F.Paste" "F.Mask")
 			(roundrect_rratio 0.25)
@@
 			(pintype "passive")
 		)
-		(model "${KICAD8_3DMODEL_DIR}/Package_TO_SOT_SMD.3dshapes/SOT-363_SC-70-6.wrl"
+		(model "${KICAD8_3DMODEL_DIR}/Package_TO_SOT_SMD.3dshapes/SOT-563.wrl"
 			(offset
 				(xyz 0 0 0)
@@
 		)
 	)
-	(footprint "Package_TO_SOT_SMD:SOT-363_SC-70-6_Handsoldering"
+	(footprint "Package_TO_SOT_SMD:SOT-563"
 		(layer "F.Cu")
 		(at 158.705002 83.199999)
-		(descr "SOT-363, SC-70-6, Handsoldering")
-		(tags "SOT-363 SC-70-6 Handsoldering")
+		(descr "SOT563")
+		(tags "SOT-563")
 		(property "Reference" "Q1"
-			(at 0 -2.25 0)
+			(at 0 -1.9 0)
 			(layer "F.SilkS")
 			(effects
@@
 		)
 		(property "Value" "DMG1024UV"
-			(at 0 2 180)
-			(layer "F.SilkS")
+			(at 0 1.75 0)
+			(layer "F.Fab")
 			(effects
 				(font
@@
 			)
 		)
-		(property "Footprint" "Package_TO_SOT_SMD:SOT-363_SC-70-6_Handsoldering"
+		(property "Footprint" "Package_TO_SOT_SMD:SOT-563"
 			(at 0 0 0)
 			(unlocked yes)
@@
 		(attr smd)
 		(fp_line
-			(start -0.71 -1.16)
-			(end 0.7 -1.16)
+			(start 0.65 -0.9)
+			(end -0.45 -0.9)
 			(stroke
 				(width 0.12)
@@
 		)
 		(fp_line
-			(start -0.7 1.16)
-			(end 0.7 1.16)
+			(start 0.65 0.9)
+			(end -0.65 0.9)
 			(stroke
 				(width 0.12)
@@
 		(fp_poly
 			(pts
-				(xy -1.08 -1.11) (xy -1.32 -1.44) (xy -0.84 -1.44) (xy -1.08 -1.11)
+				(xy -0.7 -0.9) (xy -0.98 -0.9) (xy -0.7 -1.18) (xy -0.7 -0.9)
 			)
 			(stroke
@@
 		)
 		(fp_line
-			(start -2.4 -1.4)
-			(end -2.4 1.4)
+			(start -1.35 -1.1)
+			(end -1.35 1.1)
 			(stroke
 				(width 0.05)
@@
 		)
 		(fp_line
-			(start -2.4 -1.4)
-			(end 2.4 -1.4)
+			(start -1.35 -1.1)
+			(end 1.35 -1.1)
 			(stroke
 				(width 0.05)
@@
 		)
 		(fp_line
-			(start -2.4 1.4)
-			(end 2.4 1.4)
+			(start 1.35 1.1)
+			(end -1.35 1.1)
 			(stroke
 				(width 0.05)
@@
 		)
 		(fp_line
-			(start 2.4 1.4)
-			(end 2.4 -1.4)
+			(start 1.35 1.1)
+			(end 1.35 -1.1)
 			(stroke
 				(width 0.05)
@@
 		)
 		(fp_line
-			(start -0.675 -0.6)
-			(end -0.675 1.1)
+			(start -0.65 -0.5)
+			(end -0.65 0.85)
 			(stroke
 				(width 0.1)
@@
 		)
 		(fp_line
-			(start -0.175 -1.1)
-			(end -0.675 -0.6)
+			(start -0.65 -0.5)
+			(end -0.3 -0.85)
 			(stroke
 				(width 0.1)
@@
 		)
 		(fp_line
-			(start 0.675 -1.1)
-			(end -0.175 -1.1)
+			(start -0.65 0.85)
+			(end 0.65 0.85)
 			(stroke
 				(width 0.1)
@@
 		)
 		(fp_line
-			(start 0.675 -1.1)
-			(end 0.675 1.1)
+			(start 0.65 -0.85)
+			(end -0.3 -0.85)
 			(stroke
 				(width 0.1)
@@
 		)
 		(fp_line
-			(start 0.675 1.1)
-			(end -0.675 1.1)
+			(start 0.65 0.85)
+			(end 0.65 -0.85)
 			(stroke
 				(width 0.1)
@@
 		(fp_text user "${REFERENCE}"
 			(at 0 0 90)
-			(layer "F.SilkS")
+			(layer "F.Fab")
 			(effects
 				(font
-					(size 0.5 0.5)
-					(thickness 0.075)
+					(size 0.4 0.4)
+					(thickness 0.0625)
 				)
 			)
 		)
 		(pad "1" smd roundrect
-			(at -1.33 -0.65)
-			(size 1.5 0.4)
+			(at -0.75 -0.5)
+			(size 0.7 0.34)
 			(layers "F.Cu" "F.Paste" "F.Mask")
 			(roundrect_rratio 0.25)
@@
 		)
 		(pad "2" smd roundrect
-			(at -1.33 0)
-			(size 1.5 0.4)
+			(at -0.75 0)
+			(size 0.7 0.34)
 			(layers "F.Cu" "F.Paste" "F.Mask")
 			(roundrect_rratio 0.25)
@@
 		)
 		(pad "3" smd roundrect
-			(at -1.33 0.65)
-			(size 1.5 0.4)
+			(at -0.75 0.5)
+			(size 0.7 0.34)
 			(layers "F.Cu" "F.Paste" "F.Mask")
 			(roundrect_rratio 0.25)
@@
 		)
 		(pad "4" smd roundrect
-			(at 1.33 0.65)
-			(size 1.5 0.4)
+			(at 0.75 0.5)
+			(size 0.7 0.34)
 			(layers "F.Cu" "F.Paste" "F.Mask")
 			(roundrect_rratio 0.25)
@@
 		)
 		(pad "5" smd roundrect
-			(at 1.33 0)
-			(size 1.5 0.4)
+			(at 0.75 0)
+			(size 0.7 0.34)
 			(layers "F.Cu" "F.Paste" "F.Mask")
 			(roundrect_rratio 0.25)
@@
 		)
 		(pad "6" smd roundrect
-			(at 1.33 -0.65)
-			(size 1.5 0.4)
+			(at 0.75 -0.5)
+			(size 0.7 0.34)
 			(layers "F.Cu" "F.Paste" "F.Mask")
 			(roundrect_rratio 0.25)
@@
 			(pintype "passive")
 		)
-		(model "${KICAD8_3DMODEL_DIR}/Package_TO_SOT_SMD.3dshapes/SOT-363_SC-70-6.wrl"
+		(model "${KICAD8_3DMODEL_DIR}/Package_TO_SOT_SMD.3dshapes/SOT-563.wrl"
 			(offset
 				(xyz 0 0 0)
@@
 		(tags "capacitor handsolder")
 		(property "Reference" "C22"
-			(at 0 1.429998 360)
+			(at 0 1.429998 0)
 			(layer "B.SilkS")
 			(effects
@@
 		)
 		(property "Value" "100n"
-			(at 0 -1.429998 360)
+			(at 0 -1.429998 0)
 			(layer "B.Fab")
 			(effects
@@
 		)
 		(fp_text user "${REFERENCE}"
-			(at 0 0 360)
+			(at 0 0 0)
 			(layer "B.Fab")
 			(effects
@@
 		(fp_arc
 			(start -0.675002 2.524999)
-			(mid -3.199997 -0.000001)
+			(mid -3.199996 -0.000001)
 			(end -0.675001 -2.525)
 			(stroke

Commit message: [06-05-1334] update after stagnate
Parts:
- removed J1: USB_B_Micro, Connector_USB:USB_Mini-B_Wuerth_65100516121_Horizontal
- removed J6: PORTC, Connector_PinHeader_1.27mm:PinHeader_1x16_P1.27mm_Horizontal
- C22, P1, R23, R24, SW1, U4: moved to F.Cu
- J2, J3, J4, J5: moved to B.Cu
- moved J3 43.9 mm to (161.8, 100.5), turned to 0 degrees
- moved SW1 31.7 mm to (134.0, 108.0)
- moved C19 30.7 mm to (170.0, 96.5), turned to -90 degrees
- moved D4 29.9 mm to (130.0, 96.3), turned to 90 degrees
- moved J5 29.9 mm to (154.8, 88.1), turned to 0 degrees
- moved R13 28.5 mm to (168.0, 96.5), turned to 90 degrees
- moved D3 28.3 mm to (132.0, 96.3), turned to 90 degrees
- moved R14 27.8 mm to (140.7, 107.5), turned to -90 degrees
- moved R7 27.6 mm to (132.7, 88.0)
- moved Q2 27.4 mm to (132.7, 85.9)
- moved D2 27.0 mm to (134.0, 96.3), turned to 90 degrees
- moved R12 26.6 mm to (166.0, 96.5), turned to -90 degrees
- moved D1 25.8 mm to (136.0, 96.3), turned to 90 degrees
- moved R22 25.8 mm to (130.0, 92.5), turned to 90 degrees
- moved C15 25.7 mm to (146.0, 104.2), turned to 180 degrees
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Connections:
- U3 pad 10: Net-(J6-Pin_3) -> unconnected-(U3-PC2-Pad10)
- U3 pad 11: Net-(J6-Pin_4) -> unconnected-(U3-PC3-Pad11)
- U3 pad 2: Net-(J6-Pin_14) -> unconnected-(U3-PC13-Pad2)
- U3 pad 24: Net-(J6-Pin_5) -> unconnected-(U3-PC4-Pad24)
- U3 pad 25: Net-(J6-Pin_6) -> unconnected-(U3-PC5-Pad25)
- U3 pad 3: Net-(J6-Pin_15) -> unconnected-(U3-PC14-Pad3)
- U3 pad 37: Net-(J6-Pin_7) -> unconnected-(U3-PC6-Pad37)
- U3 pad 38: Net-(J6-Pin_8) -> unconnected-(U3-PC7-Pad38)
- U3 pad 39: Net-(J6-Pin_9) -> unconnected-(U3-PC8-Pad39)
- U3 pad 4: Net-(J6-Pin_16) -> unconnected-(U3-PC15-Pad4)
- U3 pad 40: Net-(J6-Pin_10) -> unconnected-(U3-PC9-Pad40)
- U3 pad 51: Net-(J6-Pin_11) -> unconnected-(U3-PC10-Pad51)
- U3 pad 52: Net-(J6-Pin_12) -> unconnected-(U3-PC11-Pad52)
- U3 pad 53: Net-(J6-Pin_13) -> unconnected-(U3-PC12-Pad53)
- U3 pad 8: Net-(J6-Pin_1) -> unconnected-(U3-PC0-Pad8)
- U3 pad 9: Net-(J6-Pin_2) -> unconnected-(U3-PC1-Pad9)
Routing:
- net Net-(J6-Pin_5): track 62.3 -> 0.00 mm, vias 6 -> 0
- net Net-(J6-Pin_6): track 60.4 -> 0.00 mm, vias 3 -> 0
- net ITMS_DIR: track 53.7 -> 0.00 mm, vias 4 -> 0
- net GND: track 40.0 -> 92.4 mm, vias 15 -> 0
- net /TRSWO: track 47.0 -> 0.00 mm, vias 2 -> 0
- net +3.3V: track 35.9 -> 78.3 mm, vias 10 -> 0
- net ITDO: track 38.2 -> 0.00 mm, vias 2 -> 0
- net /BOOT0: track 33.9 -> 0.00 mm, vias 1 -> 0
- net /USB+: track 33.0 -> 0.00 mm, vias 2 -> 0
- net IRST_SENSE: track 32.6 -> 0.00 mm, vias 4 -> 0
- net /USB-: track 29.6 -> 0.00 mm, vias 2 -> 0
- net /SWCLK: track 28.2 -> 0.00 mm, vias 3 -> 0
- net /SWDIO: track 27.1 -> 0.00 mm, vias 1 -> 0
- net Net-(U3-PA8): track 25.8 -> 0.00 mm, vias 2 -> 0
- net PWR_BRKOUT: track 25.4 -> 0.00 mm, vias 4 -> 0
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