File: black-magic-103rc.kicad_sch (KiCad schematic)
At the start: 40 parts, among them J1 USB_B_Micro, Q1 DMG1024UV, Q2 DMG1023UV, SW1 SW_SPST, U1 USBLC6-2P6, U2 SN74LVC2T45DCUR, U3 STM32F103RCTx, U4 AMS1117-3.3, U5 SN74LVC2T45DCUR, U6 SN74LVC2T45DCUR, U7 SN74LVC2T45DCUR, Y1 8MHz

Commit message: [01-17-1939] copied schematic from reference, need to re-confirm
Update README.md
Parts:
- added C19: 100n, symbol Device:C
- added J2: Conn_ARM_JTAG_SWD_10, Connector_PinHeader_1.27mm:PinHeader_2x05_P1.27mm_Horizontal, symbol Connector:Conn_ARM_JTAG_SWD_10
- added J3: Conn_01x04, symbol Connector_Generic:Conn_01x04
- added J4, J5: Conn_01x03, symbol Connector_Generic:Conn_01x03
- added JP1: SolderJumper_2_Open, symbol Jumper:SolderJumper_2_Open
- added R10, R9: 22, symbol Device:R_US
- added R11: 1k5, symbol Device:R_US
- added R12: 4k7, symbol Device:R_US
- added R13, R14, R7, R8: 10k, symbol Device:R_US
- added RN1, RN2: 100, Resistor_SMD:R_Array_Convex_4x1206, symbol Device:R_Pack04_Split
Connections:
- net +3.3V: now also C12.1, C14.1, Q2.6 (D), U2.5 (DIR), U3.56 (PB4), U3.57 (PB5), U3.58 (PB6), U5.5 (DIR), J5.1 (Pin_1), R14.1; no longer C15.1, C16.1
- net GND: now also Q1.1 (S), Q1.4 (S), SW1.1 (A), U2.2 (A1), U2.7 (B1), U6.5 (DIR), U7.2 (A1), U7.7 (B1), Y1.2, C19.2, J2.3 (GND), J2.5 (GND), J2.9 (GNDDetect), J3.4 (Pin_4), J4.3 (Pin_3), J5.3 (Pin_3), R13.1
- net ITCK: now reaches U5.2 (A1)
- net ITCK: now also U3.21 (PA5)
- net ITDI: now reaches U5.3 (A2)
- net ITDI: now also U3.17 (PA3)
- net XTDI: now reaches U5.6 (B2)
- net XTDI: now also RN1.8 (R1.2)
- net XTCK: now reaches U5.7 (B1)
- net XTCK: now also RN2.2 (R2.1)
- net XPWR_JTAG: now reaches U5.8 (VCCB)
- net XPWR_JTAG: now also C15.1, C16.1, C17.1, C18.1, U2.8 (VCCB), U6.8 (VCCB), U7.8 (VCCB), R8.2, RN1.2 (R2.1); no longer C14.1
- net ITDO: now reaches U6.2 (A1)
- net ITDO: now also U3.22 (PA6), JP1.2 (B)
- net IRXD: now reaches U6.3 (A2)
- net IRXD: now also U3.43 (PA10)
- net XRXD: now reaches U6.6 (B2)
- net XRXD: now also RN1.3 (R3.1)
- net XTDO: now reaches U6.7 (B1)
- net XTDO: now also RN2.4 (R4.1)
- net ITMS_DIR: now reaches U3.15 (PA1)
- net ITMS_DIR: now also U7.5 (DIR)
- net IRST: now reaches U3.16 (PA2)
- net IRST: now also Q1.2 (G)
- net ITMS: now reaches U3.20 (PA4)
- net ITMS: now also U7.3 (A2)
- net IRST_SENSE: now reaches U3.23 (PA7)
- net IRST_SENSE: now also Q1.3 (D)
- net FILTERED_JTAG_PWR: now reaches U3.26 (PB0)
- net FILTERED_JTAG_PWR: now also C19.1, R12.1, R13.2
- net PWR_BRKOUT: now reaches U3.27 (PB1)
- net PWR_BRKOUT: now also Q2.2 (G), Q2.5 (G), R7.1
- net LED0: now reaches U3.28 (PB2)
- net LED0: now also R4.1
- net LED1: now reaches U3.29 (PB10)
- net LED1: now also R3.1
- net LED2: now reaches U3.30 (PB11)
- net LED2: now also R2.1
- net at U3.33 (PB12): now also SW1.2 (B), R14.2
- net VBUS: now reaches U3.34 (PB13)
- net VBUS: now also R5.1, R6.2
- net at U3.41 (PA8): now also R11.2
- net ITXD: now reaches U3.42 (PA9)
- net ITXD: now also U2.3 (A2)
- net USB-: now reaches U3.44 (PA11)
- net USB-: now also R10.2
- net USB+: now reaches U3.45 (PA12)
- net USB+: now also R9.2
- net SWDIO: now reaches U3.46 (PA13)
- net SWDIO: now also J4.1 (Pin_1)
- net SWCLK: now reaches U3.49 (PA14)
- net SWCLK: now also J4.2 (Pin_2)
- net at U3.5 (PD0): now also Y1.1
- net TDO: now reaches U3.55 (PB3)
- net TDO: now also J2.6 (SWO/TDO), RN2.5 (R4.2)
- net TRSWO: now reaches U3.59 (PB7)
- net TRSWO: now also JP1.1 (A)
- net at U3.6 (PD1): now also Y1.3
- net BOOT0: now reaches U3.60 (BOOT0)
- net BOOT0: now also J5.2 (Pin_2)
- net RST: now reaches U3.7 (NRST)
- net RST: now also J2.10 (~{RESET}), RN2.1 (R1.1)
- net PWR_JTAG: now reaches Q2.3 (D)
- net PWR_JTAG: now also J2.1 (VTref), J3.1 (Pin_1), R12.2, RN1.7 (R2.2)
- net at Q2.4 (S): now also Q2.1 (S), R7.2
- net XTXD: now reaches U2.6 (B2)
- net XTXD: now also RN1.4 (R4.1)
- net XTMS: now reaches U7.6 (B2)
- net XTMS: now also RN2.3 (R3.1)
- net XRST: now reaches Q1.5 (G)
- net XRST: now also Q1.6 (D), R8.1, RN2.8 (R1.2)
- net at U1.4 (I/O2): now also R10.1
- net at U1.6 (I/O1): now also R11.1, R9.1
- new net: J3.2 (Pin_2), RN1.5 (R4.2)
- new net: J3.3 (Pin_3), RN1.6 (R3.2)
- new net TCK: J2.4 (SWCLK/TCK), RN2.7 (R2.2)
- new net TDI: J2.8 (NC/TDI), RN1.1 (R1.1)
- new net TMS: J2.2 (SWDIO/TMS), RN2.6 (R3.2)
- no-connect marks 0 -> 9
Other:
- moved on the sheet: C1, C10, C2, C3, C4, C5, C6, C7, C8, C9, D1, D2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

Commit message: [01-19-2111] finish basic board component placement
nit
Parts:
- removed RN1, RN2: 100, Resistor_SMD:R_Array_Convex_4x1206, symbol Device:R_Pack04_Split
- removed Y1: 8MHz, symbol Device:Crystal_GND2_Small
- added C20, C21: 20p, Capacitor_SMD:C_0603_1608Metric_Pad1.08x0.95mm_HandSolder, symbol Device:C
- added R15, R16, R17, R18: 100, Resistor_SMD:R_0805_2012Metric_Pad1.20x1.40mm_HandSolder, symbol Device:R_US
- added R19, R20, R21, R22: 330, Resistor_SMD:R_0805_2012Metric_Pad1.20x1.40mm_HandSolder, symbol Device:R_US
- added Y2: 8Mhz, Crystal:Crystal_HC18-U_Vertical, symbol Device:Crystal
- C1, C10, C11, C12, C13, C14, C15, C16, C17, C18, C19, C2, C3, C4, C5, C6, C7, C8, C9: footprint (none) -> Capacitor_SMD:C_0603_1608Metric_Pad1.08x0.95mm_HandSolder
- D1, D2, D3, D4: footprint (none) -> LED_SMD:LED_0805_2012Metric_Pad1.15x1.40mm_HandSolder
- J2: value Conn_ARM_JTAG_SWD_10 -> JTAG_SWD_10; footprint Connector_PinHeader_1.27mm:PinHeader_2x05_P1.27mm_Horizontal -> Connector_PinHeader_2.54mm:PinHeader_2x05_P2.54mm_Horizontal
- J3: value Conn_01x04 -> UART; footprint (none) -> Connector_PinHeader_2.54mm:PinHeader_1x04_P2.54mm_Vertical
- J4: value Conn_01x03 -> SWD_CONN; footprint (none) -> Connector_PinHeader_2.54mm:PinHeader_1x03_P2.54mm_Vertical
- J5: value Conn_01x03 -> BOOT0; footprint (none) -> Connector_PinHeader_2.54mm:PinHeader_1x03_P2.54mm_Vertical
- JP1: value SolderJumper_2_Open -> TRSWO; footprint (none) -> Jumper:SolderJumper-2_P1.3mm_Open_RoundedPad1.0x1.5mm
- Q1: footprint (none) -> Package_TO_SOT_SMD:SOT-363_SC-70-6_Handsoldering
- R1, R2, R3, R4: value 330 -> 100; footprint (none) -> Resistor_SMD:R_0805_2012Metric_Pad1.20x1.40mm_HandSolder
- R10, R11, R12, R13, R14, R5, R6, R7, R8, R9: footprint (none) -> Resistor_SMD:R_0805_2012Metric_Pad1.20x1.40mm_HandSolder
- SW1: footprint (none) -> Button_Switch_SMD:SW_Push_1P1T_NO_6x6mm_H9.5mm
Connections:
- net +3.3V: now also R19.2; no longer R1.1
- net GND: now also C20.2, C21.2
- net LED0: now also R22.2; no longer R4.1
- net LED1: now also R21.2; no longer R3.1
- net LED2: now also R20.2; no longer R2.1
- net PWR_JTAG: now also R3.2
- net RST: now also R4.2
- net TCK: now also R15.2
- net TDI: now also R18.2
- net TDO: now also R17.2
- net TMS: now also R16.2
- net XPWR_JTAG: now also R3.1
- net XRST: now also R4.1
- net XRXD: now also R2.1
- net XTCK: now also R15.1
- net XTDI: now also R18.1
- net XTDO: now also R17.1
- net XTMS: now also R16.1
- net XTXD: now also R1.1
- net at D3.2 (A): now also R21.1; no longer R3.2
- net at U3.5 (PD0): now also C20.1, Y2.1
- net at U3.6 (PD1): now also C21.1, Y2.2
- net at R1.2: now also J3.2 (Pin_2); no longer D1.2 (A)
- net at R2.2: now also J3.3 (Pin_3); no longer D2.2 (A)
- net at D4.2 (A): now also R22.1; no longer R4.2
- new net: D1.2 (A), R19.1
- new net: D2.2 (A), R20.1
- no-connect marks 9 -> 23
Other:
- note added: "74LVC2T45"
- note added: "Indicator"
- note added: "JTAG Connector"
- note added: "STM32F103RCTx"
- note added: "Voltage Regulator"
- moved on the sheet: C1, C2, C3, D1, D2, D3, D4, U4

Commit message: [02-04-1948] start to routing
Parts:
- added C22: 100n, Capacitor_SMD:C_0603_1608Metric_Pad1.08x0.95mm_HandSolder, symbol Device:C
- added J6: PORTC, Connector_PinHeader_1.27mm:PinHeader_1x16_P1.27mm_Horizontal, symbol Connector_Generic:Conn_01x16
- added P1: USB_C_Plug_USB2.0, Connector_USB:USB_C_Receptacle_GCT_USB4110, symbol Connector:USB_C_Plug_USB2.0
- added R23, R24: 5k1, Resistor_SMD:R_0805_2012Metric_Pad1.20x1.40mm_HandSolder, symbol Device:R_US
Connections:
- net +5V: now also C22.1, P1.A4 (VBUS), P1.A9 (VBUS), P1.B4 (VBUS), P1.B9 (VBUS)
- net GND: now also C22.2, P1.A1 (GND), P1.A12 (GND), P1.B1 (GND), P1.B12 (GND), P1.S1 (SHIELD), R23.1, R24.1
- net at U3.10 (PC2): now also J6.3 (Pin_3)
- net at U3.11 (PC3): now also J6.4 (Pin_4)
- net at U3.2 (PC13): now also J6.14 (Pin_14)
- net at U3.24 (PC4): now also J6.5 (Pin_5)
- net at U3.25 (PC5): now also J6.6 (Pin_6)
- net at U3.3 (PC14): now also J6.15 (Pin_15)
- net at U3.37 (PC6): now also J6.7 (Pin_7)
- net at U3.38 (PC7): now also J6.8 (Pin_8)
- net at U3.39 (PC8): now also J6.9 (Pin_9)
- net at U3.4 (PC15): now also J6.16 (Pin_16)
- net at U3.40 (PC9): now also J6.10 (Pin_10)
- net at U3.51 (PC10): now also J6.11 (Pin_11)
- net at U3.52 (PC11): now also J6.12 (Pin_12)
- net at U3.53 (PC12): now also J6.13 (Pin_13)
- net at U3.8 (PC0): now also J6.1 (Pin_1)
- net at U3.9 (PC1): now also J6.2 (Pin_2)
- net D+: now reaches J1.3 (D+), U1.1 (I/O1)
- net D+: now also P1.A6 (D+)
- net D-: now reaches J1.2 (D-), U1.3 (I/O2)
- net D-: now also P1.A7 (D-)
- new net: P1.A5 (CC), R23.2
- new net: P1.B5 (VCONN), R24.2
- no-connect marks 23 -> 7
Other:
- moved on the sheet: C20, C21, J3, J5, R1, R2, R5, R6, Y2

Commit message: [05-25-1348] generate bom
Parts:
- Q1, Q2: footprint Package_TO_SOT_SMD:SOT-363_SC-70-6_Handsoldering -> Package_TO_SOT_SMD:SOT-563
Changed lines of the file:
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@@
 			)
 		)
-		(property "Footprint" "Package_TO_SOT_SMD:SOT-363_SC-70-6_Handsoldering"
+		(property "Footprint" "Package_TO_SOT_SMD:SOT-563"
 			(at 217.17 45.72 0)
 			(effects
@@
 			)
 		)
-		(property "Footprint" "Package_TO_SOT_SMD:SOT-363_SC-70-6_Handsoldering"
+		(property "Footprint" "Package_TO_SOT_SMD:SOT-563"
 			(at 224.79 45.72 0)
 			(effects
@@
 			)
 		)
-		(property "Footprint" "Package_TO_SOT_SMD:SOT-363_SC-70-6_Handsoldering"
+		(property "Footprint" "Package_TO_SOT_SMD:SOT-563"
 			(at 138.43 58.42 0)
 			(effects
@@
 			)
 		)
-		(property "Footprint" "Package_TO_SOT_SMD:SOT-363_SC-70-6_Handsoldering"
+		(property "Footprint" "Package_TO_SOT_SMD:SOT-563"
 			(at 138.43 58.42 0)
 			(effects

Commit message: [06-05-1334] update after stagnate
Parts:
- removed J1: USB_B_Micro, Connector_USB:USB_Mini-B_Wuerth_65100516121_Horizontal, symbol Connector:USB_B_Micro
- removed J6: PORTC, Connector_PinHeader_1.27mm:PinHeader_1x16_P1.27mm_Horizontal, symbol Connector_Generic:Conn_01x16
Other:
- moved on the sheet: J4, R10, R11, R5, R6, R9, U1
